Commit message: Add files via upload

File: baxter_description/urdf/baxter.urdf.xacro (robot description, xacro)
@@ -23,8 +23,8 @@
       <xacro:arg name="right_electric_gripper" value="${right_electric_gripper}"/>
   </xacro:include>
-  <!-- Kinect Camera -->
+  <!-- Kinect Camera for GAZEBO -->
   <xacro:include filename="$(find baxter_description)/urdf/sensors/kinect_camera.urdf.xacro"/>
-  <xacro:kinect_camera name = "kinect_camera" parent = "head">
+  <xacro:kinect_camera_gazebo name = "kinect_camera_gazebo" parent = "head">
       <origin xyz="0 0 0.1" rpy="0 0 0" />
-  </xacro:kinect_camera>
+  </xacro:kinect_camera_gazebo>
 </robot>

File: baxter_description/urdf/sensors/kinect_camera.gazebo.xacro (robot description, xacro)
@@ -5,5 +5,5 @@
       xmlns:xacro="http://www.ros.org/wiki/xacro">
 <xacro:property name="M_PI" value="3.1415926535897931" />
-<xacro:macro name="kinect_camera" params="name">
+<xacro:macro name="kinect_camera_gazebo" params="name parent *origin">
   <gazebo reference="${name}_link">
   <sensor type="depth" name="${name}_depth_frame_sensor">

File: baxter_description/urdf/sensors/kinect_camera.urdf.xacro (robot description, xacro)
@@ -26,4 +26,5 @@
       </visual>
     </link>
+	<xacro:kinect_camera_gazebo name="${name}" />
   </xacro:macro>
 </root>
